Commit message: Primera version del ROMERIN terminada.

File: romerin_description/urdf/cuerpo.xacro (robot description, xacro)
@@ -1,25 +1,22 @@
 <?xml version="1.0" ?>
 <robot name="cuerpo" xmlns:xacro="http://www.ros.org/wiki/xacro">
-<!--xacro:include filename="$(find romerin_description)/urdf/materials.xacro" /-->
-<xacro:include filename="$(find romerin_description)/urdf/cuerpo.trans" />
-<xacro:include filename="$(find romerin_description)/urdf/cuerpo.gazebo" />
 <link name="cuerpo">
   <inertial>
-    <origin rpy="0 0 0" xyz="1.2607010642475455e-06 -1.9705023201073385e-17 0.030000000000039998"/>
-    <mass value="28.985638173838137"/>
-    <inertia ixx="0.155393" ixy="-0.0" ixz="-0.0" iyy="0.159826" iyz="-0.0" izz="0.297615"/>
+	<origin rpy="0 0 0" xyz="1.2607010642475455e-06 -1.9705023201073385e-17 0.030000000000039998"/>
+	<mass value="28.985638173838137"/>
+	<inertia ixx="0.155393" ixy="-0.0" ixz="-0.0" iyy="0.159826" iyz="-0.0" izz="0.297615"/>
   </inertial>
   <visual>
-    <origin rpy="0 0 0" xyz="0 0 0"/>
-    <geometry>
-      <mesh filename="package://romerin_description/meshes/cuerpo/cuerpo.stl" scale="0.001 0.001 0.001"/>
-    </geometry>
-    <material name="silver"/>
+	<origin rpy="0 0 0" xyz="0 0 0"/>
+	<geometry>
+	  <mesh filename="package://romerin_description/meshes/cuerpo.stl" scale="0.001 0.001 0.001"/>
+	</geometry>
+	<material name="silver"/>
   </visual>
   <collision>
-    <origin rpy="0 0 0" xyz="0 0 0"/>
-    <geometry>
-      <mesh filename="package://romerin_description/meshes/cuerpo/cuerpo.stl" scale="0.001 0.001 0.001"/>
-    </geometry>
+	<origin rpy="0 0 0" xyz="0 0 0"/>
+	<geometry>
+	  <mesh filename="package://romerin_description/meshes/cuerpo.stl" scale="0.001 0.001 0.001"/>
+	</geometry>
   </collision>
 </link>

File: romerin_description/urdf/macros.xacro (robot description, xacro)
@@ -3,4 +3,5 @@
 	<xacro:macro name="body" params="parent child">
 		<joint name="fixed" type="fixed">
+  			<origin rpy="0 0 0" xyz="0 0 0.1"/>
     		<parent link="${parent}"/>
     	    <child link="${child}"/>

File: romerin_description/urdf/materials.xacro (robot description, xacro)
@@ -4,27 +4,3 @@
   <color rgba="0.700 0.700 0.700 1.000"/>
 </material>
-<material name="black">
-  <color rgba="0.0 0.0 0.0 1.0"/>
-</material>
-<material name="blue">
-  <color rgba="0.0 0.0 0.8 1.0"/>
-</material>
-<material name="green">
-  <color rgba="0.0 0.8 0.0 1.0"/>
-</material>
-<material name="grey">
-  <color rgba="0.2 0.2 0.2 1.0"/>
-</material>
-<material name="orange">
-  <color rgba="${255/255} ${108/255} ${10/255} 1.0"/>
-</material>
-<material name="brown">
-  <color rgba="${222/255} ${207/255} ${195/255} 1.0"/>
-</material>
-<material name="red">
-  <color rgba="0.8 0.0 0.0 1.0"/>
-</material>
-<material name="white">
-  <color rgba="1.0 1.0 1.0 1.0"/>
-</material>
 </robot>

File: romerin_description/urdf/pata.xacro (robot description, xacro)
@@ -1,470 +1,558 @@
 <?xml version="1.0" ?>
 <robot name="pata" xmlns:xacro="http://www.ros.org/wiki/xacro">
-<!--xacro:include filename="$(find romerin_description)/urdf/materials.xacro" /-->
-<xacro:include filename="$(find romerin_description)/urdf/pata.trans" />
-<xacro:include filename="$(find romerin_description)/urdf/pata.gazebo" />
-<xacro:macro name="pata" params="number lr">
-	<!--number: número de pata; lr: izquierda o derecha -->
+<!--xacro:include filename="$(find patacuerpo_description)/urdf/patacuerpo.trans" /-->
+<xacro:property name="PI" value="3.1415926535897931"/>
+<xacro:macro name="pata" params="lr num">
+	<!--lr: izda o dcha; num: n de pata-->
+<link name="enganche_${lr}_${num}">
+  <inertial>
+	<origin rpy="0 0 0" xyz="-0.0008835638202414636 -0.023026438950210004 7.162326287613041e-14"/>
+	<mass value="0.6779958201620729"/>
+	<inertia ixx="0.000178" ixy="2e-06" ixz="-0.0" iyy="0.000263" iyz="0.0" izz="0.000323"/>
+  </inertial>
+  <visual>
+	<origin rpy="0 0 0" xyz="-7.5e-05 0.119 -0.03"/>
+	<geometry>
+	  <mesh filename="package://patacuerpo_description/meshes/enganche_1.stl" scale="0.001 0.001 0.001"/>
+	</geometry>
+	<material name="silver"/>
+  </visual>
+  <collision>
+	<origin rpy="0 0 0" xyz="-7.5e-05 0.119 -0.03"/>
+	<geometry>
+	  <mesh filename="package://patacuerpo_description/meshes/enganche_1.stl" scale="0.001 0.001 0.001"/>
+	</geometry>
+  </collision>
+</link>
+<link name="Component2_${lr}_${num}">
+  <inertial>
+	<origin rpy="0 0 0" xyz="-3.327743548876133e-06 -0.003686600354462388 -0.0006153217354371195"/>
+	<mass value="0.04057327410573066"/>
+	<inertia ixx="3e-06" ixy="-0.0" ixz="0.0" iyy="8e-06" iyz="-0.0" izz="6e-06"/>
+  </inertial>
+  <visual>
+	<origin rpy="0 0 0" xyz="-0.015325 0.1662 -0.03"/>
+	<geometry>
+	  <mesh filename="package://patacuerpo_description/meshes/Component2_1.stl" scale="0.001 0.001 0.001"/>
+	</geometry>
+	<material name="silver"/>
+  </visual>
+  <collision>
+	<origin rpy="0 0 0" xyz="-0.015325 0.1662 -0.03"/>
+	<geometry>
+	  <mesh filename="package://patacuerpo_description/meshes/Component2_1.stl" scale="0.001 0.001 0.001"/>
+	</geometry>
+  </collision>
+</link>
+<link name="Component3_${lr}_${num}">
+  <inertial>
+	<origin rpy="0 0 0" xyz="0.017082566975035966 -0.030175162564449715 -0.011000062135107003"/>
+	<mass value="0.5890018112407169"/>
+	<inertia ixx="0.000207" ixy="-3e-06" ixz="-0.0" iyy="0.000143" iyz="-0.0" izz="0.000248"/>
+  </inertial>
+  <visual>
+	<origin rpy="0 0 0" xyz="0.001664 0.1762 -0.041"/>
+	<geometry>
+	  <mesh filename="package://patacuerpo_description/meshes/Component3_1.stl" scale="0.001 0.001 0.001"/>
+	</geometry>
+	<material name="silver"/>
+  </visual>
+  <collision>
+	<origin rpy="0 0 0" xyz="0.001664 0.1762 -0.041"/>
+	<geometry>
+	  <mesh filename="package://patacuerpo_description/meshes/Component3_1.stl" scale="0.001 0.001 0.001"/>
+	</geometry>
+  </collision>
+</link>
+<link name="Component4_${lr}_${num}">
+  <inertial>
+	<origin rpy="0 0 0" xyz="0.023500272152248945 -0.02564620791836894 -1.8395030568219006e-09"/>
+	<mass value="0.05208378573426527"/>
+	<inertia ixx="1.3e-05" ixy="0.0" ixz="0.0" iyy="2.6e-05" iyz="-0.0" izz="2.7e-05"/>
+  </inertial>
+  <visual>
+	<origin rpy="0 0 0" xyz="0.008164 0.2215 -0.03"/>
+	<geometry>
+	  <mesh filename="package://patacuerpo_description/meshes/Component4_1.stl" scale="0.001 0.001 0.001"/>
+	</geometry>
+	<material name="silver"/>
+  </visual>
+  <collision>
+	<origin rpy="0 0 0" xyz="0.008164 0.2215 -0.03"/>
+	<geometry>
+	  <mesh filename="package://patacuerpo_description/meshes/Component4_1.stl" scale="0.001 0.001 0.001"/>
+	</geometry>
+  </collision>
+</link>
+<link name="Component5_${lr}_${num}">
+  <inertial>
+	<origin rpy="0 0 0" xyz="2.7321655199363803e-07 -0.010353792081704394 7.750037417375566e-10"/>
+	<mass value="0.05208378573425636"/>
+	<inertia ixx="2.7e-05" ixy="-0.0" ixz="-0.0" iyy="2.6e-05" iyz="-0.0" izz="1.3e-05"/>
+  </inertial>
+  <visual>
+	<origin rpy="0 0 0" xyz="-0.015336 0.2575 -0.03"/>
+	<geometry>
+	  <mesh filename="package://patacuerpo_description/meshes/Component5_1.stl" scale="0.001 0.001 0.001"/>
+	</geometry>
+	<material name="silver"/>
+  </visual>
+  <collision>
+	<origin rpy="0 0 0" xyz="-0.015336 0.2575 -0.03"/>
+	<geometry>
+	  <mesh filename="package://patacuerpo_description/meshes/Component5_1.stl" scale="0.001 0.001 0.001"/>
+	</geometry>
+  </collision>
+</link>
+<link name="Component6_${lr}_${num}">
+  <inertial>
+	<origin rpy="0 0 0" xyz="2.7175869793220897e-07 -0.015124778672136407 -0.023582296616284523"/>
+	<mass value="0.5890018112407189"/>
+	<inertia ixx="0.000248" ixy="0.0" ixz="0.0" iyy="0.000143" iyz="-3e-06" izz="0.000207"/>
+  </inertial>
+  <visual>
+	<origin rpy="0 0 0" xyz="-0.015336 0.2935 -0.0535"/>
+	<geometry>
+	  <mesh filename="package://patacuerpo_description/meshes/Component6_1.stl" scale="0.001 0.001 0.001"/>
+	</geometry>
+	<material name="silver"/>
+  </visual>
+  <collision>
+	<origin rpy="0 0 0" xyz="-0.015336 0.2935 -0.0535"/>
+	<geometry>
+	  <mesh filename="package://patacuerpo_description/meshes/Component6_1.stl" scale="0.001 0.001 0.001"/>
+	</geometry>
+  </collision>
+</link>
+<link name="Component7_${lr}_${num}">
+  <inertial>
+	<origin rpy="0 0 0" xyz="0.009679299327890243 -0.13369995640458926 0.016988725070571378"/>
+	<mass value="0.8047904243141957"/>
+	<inertia ixx="0.010342" ixy="-0.0" ixz="0.0" iyy="0.000455" iyz="0.0" izz="0.010228"/>
+  </inertial>
+  <visual>
+	<origin rpy="0 0 0" xyz="-0.004336 0.3388 -0.013"/>
+	<geometry>
+	  <mesh filename="package://patacuerpo_description/meshes/Component7_1.stl" scale="0.001 0.001 0.001"/>
+	</geometry>
+	<material name="silver"/>
+  </visual>
+  <collision>
+	<origin rpy="0 0 0" xyz="-0.004336 0.3388 -0.013"/>
+	<geometry>
+	  <mesh filename="package://patacuerpo_description/meshes/Component7_1.stl" scale="0.001 0.001 0.001"/>
+	</geometry>
+  </collision>
+</link>
+<link name="Component8_${lr}_${num}">
+  <inertial>
+	<origin rpy="0 0 0" xyz="0.024875371372866634 -0.017300001288044542 -0.017039615317225636"/>
+	<mass value="0.5890018112407238"/>
+	<inertia ixx="0.000143" ixy="0.0" ixz="-3e-06" iyy="0.000248" iyz="-0.0" izz="0.000207"/>
+  </inertial>
+  <visual>
+	<origin rpy="0 0 0" xyz="0.002664 0.6062 -0.046977"/>
+	<geometry>
+	  <mesh filename="package://patacuerpo_description/meshes/Component8_1.stl" scale="0.001 0.001 0.001"/>
+	</geometry>
+	<material name="silver"/>
+  </visual>
+  <collision>
+	<origin rpy="0 0 0" xyz="0.002664 0.6062 -0.046977"/>
+	<geometry>
+	  <mesh filename="package://patacuerpo_description/meshes/Component8_1.stl" scale="0.001 0.001 0.001"/>
+	</geometry>
+  </collision>
+</link>
+<link name="Component9_${lr}_${num}">
+  <inertial>
+	<origin rpy="0 0 0" xyz="-0.01880335468036301 -0.030302739995931915 0.023500457245787268"/>
+	<mass value="0.07064606392588994"/>
+	<inertia ixx="5.1e-05" ixy="-5e-06" ixz="-0.0" iyy="4.1e-05" iyz="0.0" izz="2.9e-05"/>
+  </inertial>
+  <visual>
+	<origin rpy="0 0 0" xyz="-0.037336 0.6235 -0.007977"/>
+	<geometry>
+	  <mesh filename="package://patacuerpo_description/meshes/Component9_1.stl" scale="0.001 0.001 0.001"/>
+	</geometry>
+	<material name="silver"/>
+  </visual>
+  <collision>
+	<origin rpy="0 0 0" xyz="-0.037336 0.6235 -0.007977"/>
+	<geometry>
+	  <mesh filename="package://patacuerpo_description/meshes/Component9_1.stl" scale="0.001 0.001 0.001"/>
+	</geometry>
+  </collision>
+</link>
+<link name="Component10_${lr}_${num}">
+  <inertial>
+	<origin rpy="0 0 0" xyz="-0.0017135454980912197 -0.15691041401299965 -0.0007575519701589137"/>
+	<mass value="1.969918180322282"/>
+	<inertia ixx="0.021818" ixy="0.000391" ixz="3e-06" iyy="0.000894" iyz="-0.000131" izz="0.021632"/>
+  </inertial>
+  <visual>
+	<origin rpy="0 0 0" xyz="-0.015336 0.6715 -0.031477"/>
+	<geometry>
+	  <mesh filename="package://patacuerpo_description/meshes/Component10_1.stl" scale="0.001 0.001 0.001"/>
+	</geometry>
+	<material name="silver"/>
+  </visual>
+  <collision>
+	<origin rpy="0 0 0" xyz="-0.015336 0.6715 -0.031477"/>
+	<geometry>
+	  <mesh filename="package://patacuerpo_description/meshes/Component10_1.stl" scale="0.001 0.001 0.001"/>
+	</geometry>
+  </collision>
+</link>
+<link name="Component11_${lr}_${num}">
+  <inertial>
+	<origin rpy="0 0 0" xyz="0.007623821851629745 -2.9323939987335734e-07 -2.1019877097794293e-06"/>
+	<mass value="0.04831387336471295"/>
+	<inertia ixx="7e-06" ixy="-0.0" ixz="-0.0" iyy="5e-06" iyz="-0.0" izz="5e-06"/>
+  </inertial>
+  <visual>
+	<origin rpy="0 0 0" xyz="-0.0307 0.932519 -0.030023"/>
+	<geometry>
+	  <mesh filename="package://patacuerpo_description/meshes/Component11_1.stl" scale="0.001 0.001 0.001"/>
+	</geometry>
+	<material name="silver"/>
+  </visual>
+  <collision>
+	<origin rpy="0 0 0" xyz="-0.0307 0.932519 -0.030023"/>
+	<geometry>
+	  <mesh filename="package://patacuerpo_description/meshes/Component11_1.stl" scale="0.001 0.001 0.001"/>
+	</geometry>
+  </collision>
+</link>
+<link name="Component13_${lr}_${num}">
+  <inertial>
+	<origin rpy="0 0 0" xyz="-7.046964762767727e-05 -0.025651671856746106 -8.711431092059407e-06"/>
+	<mass value="0.9228320571083133"/>
+	<inertia ixx="0.00065" ixy="-1e-06" ixz="0.0" iyy="0.000398" iyz="0.0" izz="0.000533"/>
+  </inertial>
+  <visual>
+	<origin rpy="0 0 0" xyz="-0.015336 0.956561 -0.030023"/>
+	<geometry>
+	  <mesh filename="package://patacuerpo_description/meshes/Component13_1.stl" scale="0.001 0.001 0.001"/>
+	</geometry>
+	<material name="silver"/>
+  </visual>
+  <collision>
+	<origin rpy="0 0 0" xyz="-0.015336 0.956561 -0.030023"/>
+	<geometry>
+	  <mesh filename="package://patacuerpo_description/meshes/Component13_1.stl" scale="0.001 0.001 0.001"/>
+	</geometry>
+  </collision>
+</link>
+<link name="Component14_${lr}_${num}">
+  <inertial>
+	<origin rpy="0 0 0" xyz="-1.0024119439892842e-07 -1.2555316453166654e-07 -0.0016568293364659743"/>
+	<mass value="0.11553702060403329"/>
+	<inertia ixx="2.9e-05" ixy="-0.0" ixz="-0.0" iyy="2.9e-05" iyz="0.0" izz="3.6e-05"/>
+  </inertial>
+  <visual>
+	<origin rpy="0 0 0" xyz="-0.01507 1.002493 0.001477"/>
+	<geometry>
+	  <mesh filename="package://patacuerpo_description/meshes/Component14_1.stl" scale="0.001 0.001 0.001"/>
+	</geometry>
+	<material name="silver"/>
+  </visual>
+  <collision>
+	<origin rpy="0 0 0" xyz="-0.01507 1.002493 0.001477"/>
+	<geometry>
+	  <mesh filename="package://patacuerpo_description/meshes/Component14_1.stl" scale="0.001 0.001 0.001"/>
+	</geometry>
+  </collision>
+</link>
+<link name="Component17_${lr}_${num}">
+  <inertial>
+	<origin rpy="0 0 0" xyz="-1.2322251817693808e-07 0.003859592424359626 -4.557914220180981e-07"/>
+	<mass value="0.22106688110468858"/>
+	<inertia ixx="6.7e-05" ixy="0.0" ixz="-0.0" iyy="0.000129" iyz="-0.0" izz="6.7e-05"/>
+  </inertial>
+  <visual>
+	<origin rpy="0 0 0" xyz="-0.01507 1.035027 -0.030023"/>
+	<geometry>
+	  <mesh filename="package://patacuerpo_description/meshes/Component17_1.stl" scale="0.001 0.001 0.001"/>
+	</geometry>
+	<material name="silver"/>
+  </visual>
+  <collision>
+	<origin rpy="0 0 0" xyz="-0.01507 1.035027 -0.030023"/>
+	<geometry>
+	  <mesh filename="package://patacuerpo_description/meshes/Component17_1.stl" scale="0.001 0.001 0.001"/>
+	</geometry>
+  </collision>
+</link>
+<link name="Component12_${lr}_${num}">
+  <inertial>
+	<origin rpy="0 0 0" xyz="-0.0018786122979095599 3.870314608800385e-07 1.0481699663222876e-06"/>
+	<mass value="0.044964172872987526"/>
+	<inertia ixx="7e-06" ixy="0.0" ixz="-0.0" iyy="4e-06" iyz="0.0" izz="4e-06"/>
+  </inertial>
+  <visual>
+	<origin rpy="0 0 0" xyz="0.007027 0.932502 -0.030032"/>
+	<geometry>
+	  <mesh filename="package://patacuerpo_description/meshes/Component12_1.stl" scale="0.001 0.001 0.001"/>
+	</geometry>
+	<material name="silver"/>
+  </visual>
+  <collision>
+	<origin rpy="0 0 0" xyz="0.007027 0.932502 -0.030032"/>
+	<geometry>
+	  <mesh filename="package://patacuerpo_description/meshes/Component12_1.stl" scale="0.001 0.001 0.001"/>
+	</geometry>
+  </collision>
+</link>
+<link name="Component15_${lr}_${num}">
+  <inertial>
+	<origin rpy="0 0 0" xyz="-9.926848198830995e-08 -7.599328972318631e-06 0.0030593073916383787"/>
+	<mass value="0.11084533748383699"/>
+	<inertia ixx="1.9e-05" ixy="0.0" ixz="0.0" iyy="1.9e-05" iyz="0.0" izz="3.6e-05"/>
+  </inertial>
+  <visual>
+	<origin rpy="0 0 0" xyz="-0.01507 1.00247 -0.061523"/>
+	<geometry>
+	  <mesh filename="package://patacuerpo_description/meshes/Component15_1.stl" scale="0.001 0.001 0.001"/>
+	</geometry>
+	<material name="silver"/>
+  </visual>
+  <collision>
+	<origin rpy="0 0 0" xyz="-0.01507 1.00247 -0.061523"/>
+	<geometry>
+	  <mesh filename="package://patacuerpo_description/meshes/Component15_1.stl" scale="0.001 0.001 0.001"/>
+	</geometry>
+  </collision>
+</link>
+<link name="Component16_${lr}_${num}">
+  <inertial>
+	<origin rpy="0 0 0" xyz="4.663110592786901e-06 -0.024171205343439528 -0.03812145579226034"/>
+	<mass value="0.07272237784571686"/>
+	<inertia ixx="8.5e-05" ixy="0.0" ixz="0.0" iyy="8.6e-05" iyz="-0.0" izz="2.6e-05"/>
+  </inertial>
+  <visual>
+	<origin rpy="0 0 0" xyz="-0.01507 1.002478 -0.068144"/>
+	<geometry>
+	  <mesh filename="package://patacuerpo_description/meshes/Component16_1.stl" scale="0.001 0.001 0.001"/>
+	</geometry>
+	<material name="silver"/>
+  </visual>
+  <collision>
+	<origin rpy="0 0 0" xyz="-0.01507 1.002478 -0.068144"/>
+	<geometry>
+	  <mesh filename="package://patacuerpo_description/meshes/Component16_1.stl" scale="0.001 0.001 0.001"/>
+	</geometry>
+  </collision>
+</link>
 	<!--Primera joint: cuerpo-pata-->
-	<joint type="fixed" name="hinge_${lr}_${number}_1">
-    	<parent link="cuerpo"/>
-    	<child link="enganche_${lr}_${number}"/>
-    	<xacro:if value="${lr == 'left'}">
-			<xacro:if value="${number == '1'}">
-      			<origin rpy="0 0 0" xyz="0.085075 0.119 0.03"/>
+<joint name="Rigid0_${lr}_${num}" type="fixed">
+  <parent link="cuerpo"/>
+  <child link="enganche_${lr}_${num}"/>
+    	<xacro:if value="${lr == 'l'}">
+			<xacro:if value="${num == 1}">
+      			<origin rpy="${PI} 0 0" xyz="0.085075 0.119 0.03"/>
 			</xacro:if>
-			<xacro:if value="${number == '2'}">
-      			<origin rpy="0 0 0" xyz="7.5e-05 0.119 0.03"/>
+			<xacro:if value="${num == 2}">
+      			<origin rpy="${PI} 0 0" xyz="7.5e-05 0.119 0.03"/>
 			</xacro:if>
-			<xacro:if value="${number == '3'}">
-      			<origin rpy="0 0 0" xyz="-0.084925 0.119 0.03"/>
+			<xacro:if value="${num == 3}">
+      			<origin rpy="${PI} 0 0" xyz="-0.084925 0.119 0.03"/>
 			</xacro:if>
     	</xacro:if>
-    	<xacro:if value="${lr == 'right'}">
-			<xacro:if value="${number == '1'}">
+    	<xacro:if value="${lr == 'r'}">
+			<xacro:if value="${num == 1}">
       			<origin rpy="0 0 0" xyz="0.085075 -0.119 0.03"/>
 			</xacro:if>
-			<xacro:if value="${number == '2'}">
-      			 <origin rpy="0 0 0" xyz="7.5e-05 -0.119 0.03"/>
+			<xacro:if value="${num == 2}">
+ 				<origin rpy="0 0 0" xyz="7.5e-05 -0.119 0.03"/>
 			</xacro:if>
-			<xacro:if value="${number == '3'}">
+			<xacro:if value="${num == 3}">
       			<origin rpy="0 0 0" xyz="-0.084925 -0.119 0.03"/>
 			</xacro:if>
     	</xacro:if>
-    	<!--limit effort="${limit_effort}" velocity="${limit_velocity}" lower="${limit_lower_1}" upper="${limit_upper_1}" /-->
-  	</joint>
-	<link name="enganche_${lr}_${number}">
-	  <inertial>
-   		<origin rpy="0 0 0" xyz="-0.0008835638202414636 -0.023026438950210004 7.162326287613041e-14"/>
-		<mass value="0.6779958201620729"/>
-        <inertia ixx="0.000178" ixy="2e-06" ixz="-0.0" iyy="0.000263" iyz="0.0" izz="0.000323"/>
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
File: romerin_description/urdf/romerin.xacro (robot description, xacro)
@@ -1,25 +1,21 @@
-<?xml version="1.0"?>
+<?xml version="1.0" ?>
 <robot name="romerin" xmlns:xacro="http://www.ros.org/wiki/xacro">
+<xacro:include filename="$(find romerin_description)/urdf/materials.xacro" />
 <xacro:include filename="$(find romerin_description)/urdf/macros.xacro" />
-<xacro:include filename="$(find romerin_description)/urdf/materials.xacro" />
+<xacro:include filename="$(find romerin_description)/urdf/pata.xacro" />
 <xacro:include filename="$(find romerin_description)/urdf/cuerpo.xacro" />
-<xacro:include filename="$(find romerin_description)/urdf/romerin.trans"/>
-<!--xacro:include filename="$(find romerin_description)/urdf/cuerpo.trans" /-->
-<!--xacro:include filename="$(find romerin_description)/urdf/cuerpo.gazebo" /-->
-<xacro:include filename="$(find romerin_description)/urdf/pata.xacro" />
-<!--xacro:include filename="$(find romerin_description)/urdf/pata.trans" /-->
-<!--xacro:include filename="$(find romerin_description)/urdf/pata.gazebo" /-->
+<xacro:include filename="$(find romerin_description)/urdf/romerin.gazebo" />
+<!--xacro:include filename="$(find romerin_description)/urdf/romerin.trans" /-->
+	<!--romerin.trans no se incluye porque su codigo se ha pegado en pata.xacro-->
 <!-- Used for fixing robot to Gazebo 'base_link (frame reference)' -->
 <link name="base_link"/>
 <!-- Body -->
 <xacro:body parent="base_link" child="cuerpo"/>
-<!-- Legs -->
-<xacro:pata number="2" lr="right"/>
-<!--
-<joint name="Romerin_rig_1" type="fixed">
-  <origin rpy="0 0 0" xyz="-0.084925 -0.119 0.03"/>
-  <parent link="cuerpo"/>
-  <child link="enganche"/>
-</joint>
--->
+<!--Legs-->
+<xacro:pata lr="r" num="1"/>
+<xacro:pata lr="r" num="2"/>
+<xacro:pata lr="r" num="3"/>
+<xacro:pata lr="l" num="1"/>
+<xacro:pata lr="l" num="2"/>
+<xacro:pata lr="l" num="3"/>
 </robot>
