Commit message: Última versión del ROMERIN y primera del Robominer.

File: robominer_description/urdf/macros.xacro (robot description, xacro)
@@ -1,4 +1,4 @@
 <?xml version="1.0"?>
-<robot name="romerin" xmlns:xacro="http://www.ros.org/wiki/xacro">
+<robot name="robominer" xmlns:xacro="http://www.ros.org/wiki/xacro">
 	<xacro:macro name="body" params="parent child">
 		<joint name="fixed" type="fixed">

File: romerin_description/urdf/pata.xacro (robot description, xacro)
@@ -373,15 +373,9 @@
 </joint>
 <joint name="Rigid1_${lr}_${num}" type="fixed">
-  <origin rpy="0 ${PI/2}  0" xyz="0.01525 -0.0472 0.0"/>
+	<xacro:if value="${lr == 'r'}">
+  		<origin rpy="0 ${PI/2}  0" xyz="0.01525 -0.0472 0.0"/>
+	</xacro:if>
 	<xacro:if value="${lr == 'l'}">
-		<xacro:if value="${num == 1}">
-			<origin rpy="0 ${3*PI/2} 0" xyz="0.01525 -0.0472 0.0"/>
-		</xacro:if>
-		<xacro:if value="${num == 2}">
-			<origin rpy="0 ${3*PI/2} 0" xyz="0.01525 -0.0472 0.0"/>
-		</xacro:if>
-		<xacro:if value="${num == 3}">
-			<origin rpy="0 ${3*PI/2} 0" xyz="0.01525 -0.0472 0.0"/>
-		</xacro:if>
+		<origin rpy="0 ${3*PI/2} 0" xyz="0.01525 -0.0472 0.0"/>
 	</xacro:if>
   <parent link="enganche_${lr}_${num}"/>
