Commit message: Solucionado el tembleque al lanzar los controladores

File: robominer_description/urdf/pata.xacro (robot description, xacro)
@@ -278,4 +278,6 @@
     	</xacro:if>
 </joint>
+	<!--Tengo que probar si colocando la siguiente etiqueta en todas las joints evito las vibraciones-->
+<!--dynamics damping="0.7" friction="100.0" /-->
 <joint name="Rigid1_${lr}_${num}" type="fixed">
   <xacro:if value="${lr == 'r'}">
@@ -298,4 +300,5 @@
   <child link="Component4_${lr}_${num}"/>
   <axis xyz="-0.0 -0.0 1.0"/>
+  <dynamics damping=".1" friction="1.0" />
   <limit effort="100" lower="-1.919862" upper="1.919862" velocity="100"/>
 </joint>
@@ -310,4 +313,5 @@
   <child link="Component6_${lr}_${num}"/>
   <axis xyz="-1.0 0.0 -0.0"/>
+  <dynamics damping=".1" friction="1.0" />
   <limit effort="100" lower="-1.919862" upper="1.919862" velocity="100"/>
 </joint>
@@ -327,4 +331,5 @@
   <child link="Component9_${lr}_${num}"/>
   <axis xyz="1.0 -0.0 0.0"/>
+  <dynamics damping=".1" friction="1.0" />
   <limit effort="100" lower="-0.785398" upper="3.141593" velocity="100"/>
 </joint>
@@ -344,4 +349,5 @@
   <child link="Component12_${lr}_${num}"/>
   <axis xyz="1.0 -0.0 0.0"/>
+  <dynamics damping=".1" friction="1.0" />
   <limit effort="100" lower="-1.570796" upper="1.570796" velocity="100"/>
 </joint>

File: robominer_description/urdf/robominer.xacro (robot description, xacro)
@@ -5,6 +5,6 @@
 <xacro:include filename="$(find robominer_description)/urdf/pata.xacro" />
 <xacro:include filename="$(find robominer_description)/urdf/cuerpo.xacro" />
-<xacro:include filename="$(find robominer_description)/urdf/robominer.gazebo" />
-<!--xacro:include filename="$(find robominer_description)/urdf/robominer_alt.gazebo" /-->
+<!--xacro:include filename="$(find robominer_description)/urdf/robominer.gazebo"/-->
+<xacro:include filename="$(find robominer_description)/urdf/robominer_alt.gazebo"/>
 <!--xacro:include filename="$(find robominer_description)/urdf/robominer.trans" /-->
 	<!--robominer.trans no se incluye porque su codigo se ha pegado en pata.xacro-->
