Commit message: Primer script de control del Robominer

File: robominer_description/urdf/cuerpo.xacro (robot description, xacro)
@@ -4,5 +4,6 @@
   <inertial>
 	<origin rpy="0 0 0" xyz="1.2607010642475455e-06 -1.9705023201073385e-17 0.030000000000039998"/>
-	<mass value="28.985638173838137"/>
+	<!--mass value="28.985638173838137"/-->
+	<mass value="2"/>
 	<inertia ixx="0.155393" ixy="-0.0" ixz="-0.0" iyy="0.159826" iyz="-0.0" izz="0.297615"/>
   </inertial>

Commit message: Pongo el repo al día con todo.

File: robominer_description/urdf/cuerpo.xacro (robot description, xacro)
@@ -22,3 +22,10 @@
   </collision>
 </link>
+<xacro:macro name="body" params="parent child">
+	<joint name="fixed" type="fixed">
+		<origin rpy="0 0 0" xyz="0 0 0.1"/>
+		<parent link="${parent}"/>
+		<child link="${child}"/>
+	</joint>
+</xacro:macro>
 </robot>

File: robominer_description/urdf/pata.xacro (robot description, xacro)
@@ -278,6 +278,4 @@
     	</xacro:if>
 </joint>
-	<!--Tengo que probar si colocando la siguiente etiqueta en todas las joints evito las vibraciones-->
-<!--dynamics damping="0.7" friction="100.0" /-->
 <joint name="Rigid1_${lr}_${num}" type="fixed">
   <xacro:if value="${lr == 'r'}">
@@ -312,5 +310,5 @@
   <parent link="Component5_${lr}_${num}"/>
   <child link="Component6_${lr}_${num}"/>
-  <axis xyz="-1.0 0.0 -0.0"/>
+  <axis xyz="1.0 0.0 -0.0"/>
   <dynamics damping=".1" friction="1.0" />
   <limit effort="100" lower="-1.919862" upper="1.919862" velocity="100"/>
@@ -330,5 +328,5 @@
   <parent link="Component8_${lr}_${num}"/>
   <child link="Component9_${lr}_${num}"/>
-  <axis xyz="1.0 -0.0 0.0"/>
+  <axis xyz="1.0 0.0 0.0"/>
   <dynamics damping=".1" friction="1.0" />
   <limit effort="100" lower="-0.785398" upper="3.141593" velocity="100"/>
@@ -396,14 +394,14 @@
 <!-- Enable the Joint Feedback -->
 <gazebo reference="Rev3_${lr}_${num}">
-<provideFeedback>true</provideFeedback>
+  <provideFeedback>true</provideFeedback>
 </gazebo>
 <!-- The ft_sensor plugin -->
 <gazebo>
-<plugin name="ft_sensor" filename="libgazebo_ros_ft_sensor.so">
-  <robotNamespace>/robominer</robotNamespace>
-<updateRate>100.0</updateRate>
-<topicName>Rev3_${lr}_${num}_ft_sensor_topic</topicName>
-<jointName>Rev3_${lr}_${num}</jointName>
-</plugin>
+  <plugin name="ft_sensor" filename="libgazebo_ros_ft_sensor.so">
+    <robotNamespace>/robominer</robotNamespace>
+	<updateRate>100.0</updateRate>
+	<topicName>Rev3_${lr}_${num}_ft_sensor_topic</topicName>
+	<jointName>Rev3_${lr}_${num}</jointName>
+  </plugin>
 </gazebo>
 <!-- Enable the Joint Feedback -->

File: robominer_description/urdf/robominer.xacro (robot description, xacro)
@@ -2,5 +2,5 @@
 <robot name="robominer" xmlns:xacro="http://www.ros.org/wiki/xacro">
 <xacro:include filename="$(find robominer_description)/urdf/materials.xacro" />
-<xacro:include filename="$(find robominer_description)/urdf/macros.xacro" />
+<!--xacro:include filename="$(find robominer_description)/urdf/macros.xacro" /-->
 <xacro:include filename="$(find robominer_description)/urdf/pata.xacro" />
 <xacro:include filename="$(find robominer_description)/urdf/cuerpo.xacro" />

Commit message: Update cuerpo.xacro

File: robominer_description/urdf/cuerpo.xacro (robot description, xacro)
@@ -1,31 +1,30 @@
 <?xml version="1.0" ?>
 <robot name="cuerpo" xmlns:xacro="http://www.ros.org/wiki/xacro">
-<link name="cuerpo">
-  <inertial>
-	<origin rpy="0 0 0" xyz="1.2607010642475455e-06 -1.9705023201073385e-17 0.030000000000039998"/>
-	<!--mass value="28.985638173838137"/-->
-	<mass value="2"/>
-	<inertia ixx="0.155393" ixy="-0.0" ixz="-0.0" iyy="0.159826" iyz="-0.0" izz="0.297615"/>
-  </inertial>
-  <visual>
-	<origin rpy="0 0 0" xyz="0 0 0"/>
-	<geometry>
-	  <mesh filename="package://robominer_description/meshes/cuerpo.stl" scale="0.001 0.001 0.001"/>
-	</geometry>
-	<material name="silver"/>
-  </visual>
-  <collision>
-	<origin rpy="0 0 0" xyz="0 0 0"/>
-	<geometry>
-	  <mesh filename="package://robominer_description/meshes/cuerpo.stl" scale="0.001 0.001 0.001"/>
-	</geometry>
-  </collision>
-</link>
-<xacro:macro name="body" params="parent child">
-	<joint name="fixed" type="fixed">
-		<origin rpy="0 0 0" xyz="0 0 0.1"/>
-		<parent link="${parent}"/>
-		<child link="${child}"/>
-	</joint>
-</xacro:macro>
+  <link name="cuerpo">
+    <inertial>
+      <origin rpy="0 0 0" xyz="1.2607010642475455e-06 -1.9705023201073385e-17 0.030000000000039998"/>
+      <mass value="2"/>
+      <inertia ixx="0.155393" ixy="-0.0" ixz="-0.0" iyy="0.159826" iyz="-0.0" izz="0.297615"/>
+    </inertial>
+    <visual>
+      <origin rpy="0 0 0" xyz="0 0 0"/>
+      <geometry>
+        <mesh filename="package://robominer_description/meshes/cuerpo.stl" scale="0.001 0.001 0.001"/>
+      </geometry>
+       <material name="silver"/>
+    </visual>
+    <collision>
+      <origin rpy="0 0 0" xyz="0 0 0"/>
+      <geometry>
+        <mesh filename="package://robominer_description/meshes/cuerpo.stl" scale="0.001 0.001 0.001"/>
+      </geometry>
+    </collision>
+  </link>
+  <xacro:macro name="body" params="parent child">
+    <joint name="fixed" type="fixed">
+      <origin rpy="0 0 0" xyz="0 0 0.1"/>
+      <parent link="${parent}"/>
+      <child link="${child}"/>
+    </joint>
+  </xacro:macro>
 </robot>

Commit message: Update cuerpo.xacro

File: robominer_description/urdf/cuerpo.xacro (robot description, xacro)
@@ -1,30 +1,74 @@
 <?xml version="1.0" ?>
 <robot name="cuerpo" xmlns:xacro="http://www.ros.org/wiki/xacro">
-  <link name="cuerpo">
-    <inertial>
-      <origin rpy="0 0 0" xyz="1.2607010642475455e-06 -1.9705023201073385e-17 0.030000000000039998"/>
-      <mass value="2"/>
-      <inertia ixx="0.155393" ixy="-0.0" ixz="-0.0" iyy="0.159826" iyz="-0.0" izz="0.297615"/>
-    </inertial>
-    <visual>
-      <origin rpy="0 0 0" xyz="0 0 0"/>
-      <geometry>
-        <mesh filename="package://robominer_description/meshes/cuerpo.stl" scale="0.001 0.001 0.001"/>
-      </geometry>
-       <material name="silver"/>
-    </visual>
-    <collision>
-      <origin rpy="0 0 0" xyz="0 0 0"/>
-      <geometry>
-        <mesh filename="package://robominer_description/meshes/cuerpo.stl" scale="0.001 0.001 0.001"/>
-      </geometry>
-    </collision>
-  </link>
-  <xacro:macro name="body" params="parent child">
-    <joint name="fixed" type="fixed">
-      <origin rpy="0 0 0" xyz="0 0 0.1"/>
-      <parent link="${parent}"/>
-      <child link="${child}"/>
-    </joint>
-  </xacro:macro>
+<link name="cuerpo">
+  <inertial>
+	<origin rpy="0 0 0" xyz="1.2607010642475455e-06 -1.9705023201073385e-17 0.030000000000039998"/>
+	<!--mass value="28.985638173838137"/-->
+	<mass value="10"/>
+	<!--mass value="2"/-->
+	<inertia ixx="0.155393" ixy="-0.0" ixz="-0.0" iyy="0.159826" iyz="-0.0" izz="0.297615"/>
+  </inertial>
+  <visual>
+	<origin rpy="0 0 0" xyz="0 0 0"/>
+	<geometry>
+	  <mesh filename="package://robominer_description/meshes/cuerpo.stl" scale="0.001 0.001 0.001"/>
+	</geometry>
+	<material name="silver"/>
+  </visual>
+  <collision>
+	<origin rpy="0 0 0" xyz="0 0 0"/>
+	<geometry>
+	  <mesh filename="package://robominer_description/meshes/cuerpo.stl" scale="0.001 0.001 0.001"/>
+	</geometry>
+  </collision>
+</link>
+<link name="logo1">
+  <visual>
+    <origin rpy="0 0 0" xyz="0 0 0"/>
+    <geometry>
+      <mesh filename="package://robominer_description/meshes/logo1.stl" scale="0.001 0.001 0.001"/>
+    </geometry>
+    <material name="logored"/>
+  </visual>
+</link>
+<link name="logo2">
+  <visual>
+    <origin rpy="0 0 0" xyz="0 0 0"/>
+    <geometry>
+      <mesh filename="package://robominer_description/meshes/logo2.stl" scale="0.001 0.001 0.001"/>
+    </geometry>
+    <material name="white"/>
+  </visual>
+</link>
+<link name="ladrilloslogo">
+  <visual>
+    <origin rpy="0 0 0" xyz="0 0 0"/>
+    <geometry>
+      <mesh filename="package://robominer_description/meshes/ladrilloslogo.stl" scale="0.001 0.001 0.001"/>
+    </geometry>
+    <material name="logored"/>
+  </visual>
+</link>
+<joint name="cuerpo_logo1" type="fixed">
+	<origin rpy="0 0 0.5236" xyz="-0.006 0.105 0.0551"/>
+	<parent link="cuerpo"/>
+	<child link="logo1"/>
+</joint>
+<joint name="cuerpo_logo2" type="fixed">
+	<origin rpy="0 0 -1.5707" xyz="0.08 0.125 0.0552"/>
+	<parent link="cuerpo"/>
+	<child link="logo2"/>
+</joint>
+<joint name="cuerpo_ladrillos" type="fixed">
+	<origin rpy="0 0 -1.5707" xyz="0.08 0.125 0.0551"/>
+	<parent link="cuerpo"/>
+	<child link="ladrilloslogo"/>
+</joint>
+<xacro:macro name="body" params="parent child">
+	<joint name="fixed" type="fixed">
+		<origin rpy="0 0 0" xyz="0 0 0.1"/>
+		<parent link="${parent}"/>
+		<child link="${child}"/>
+	</joint>
+</xacro:macro>
 </robot>

Commit message: Commit cuerpo

File: robominer_description/urdf/cuerpo.xacro (robot description, xacro)
@@ -1,9 +1,11 @@
 <?xml version="1.0" ?>
 <robot name="cuerpo" xmlns:xacro="http://www.ros.org/wiki/xacro">
+<<<<<<< HEAD
 <link name="cuerpo">
   <inertial>
 	<origin rpy="0 0 0" xyz="1.2607010642475455e-06 -1.9705023201073385e-17 0.030000000000039998"/>
 	<!--mass value="28.985638173838137"/-->
-	<mass value="2"/>
+	<mass value="10"/>
+	<!--mass value="2"/-->
 	<inertia ixx="0.155393" ixy="-0.0" ixz="-0.0" iyy="0.159826" iyz="-0.0" izz="0.297615"/>
   </inertial>
@@ -22,4 +24,46 @@
   </collision>
 </link>
+<link name="logo1">
+  <visual>
+    <origin rpy="0 0 0" xyz="0 0 0"/>
+    <geometry>
+      <mesh filename="package://robominer_description/meshes/logo1.stl" scale="0.001 0.001 0.001"/>
+    </geometry>
+    <material name="logored"/>
+  </visual>
+</link>
+<link name="logo2">
+  <visual>
+    <origin rpy="0 0 0" xyz="0 0 0"/>
+    <geometry>
+      <mesh filename="package://robominer_description/meshes/logo2.stl" scale="0.001 0.001 0.001"/>
+    </geometry>
+    <material name="white"/>
+  </visual>
+</link>
+<link name="ladrilloslogo">
+  <visual>
+    <origin rpy="0 0 0" xyz="0 0 0"/>
+    <geometry>
+      <mesh filename="package://robominer_description/meshes/ladrilloslogo.stl" scale="0.001 0.001 0.001"/>
+    </geometry>
+    <material name="logored"/>
+  </visual>
+</link>
+<joint name="cuerpo_logo1" type="fixed">
+	<origin rpy="0 0 0.5236" xyz="-0.006 0.105 0.0551"/>
+	<parent link="cuerpo"/>
+	<child link="logo1"/>
+</joint>
+<joint name="cuerpo_logo2" type="fixed">
+	<origin rpy="0 0 -1.5707" xyz="0.08 0.125 0.0552"/>
+	<parent link="cuerpo"/>
+	<child link="logo2"/>
+</joint>
+<joint name="cuerpo_ladrillos" type="fixed">
+	<origin rpy="0 0 -1.5707" xyz="0.08 0.125 0.0551"/>
+	<parent link="cuerpo"/>
+	<child link="ladrilloslogo"/>
+</joint>
 <xacro:macro name="body" params="parent child">
 	<joint name="fixed" type="fixed">
@@ -29,3 +73,32 @@
 	</joint>
 </xacro:macro>
+=======
+  <link name="cuerpo">
+    <inertial>
+      <origin rpy="0 0 0" xyz="1.2607010642475455e-06 -1.9705023201073385e-17 0.030000000000039998"/>
+      <mass value="2"/>
+      <inertia ixx="0.155393" ixy="-0.0" ixz="-0.0" iyy="0.159826" iyz="-0.0" izz="0.297615"/>
+    </inertial>
+    <visual>
+      <origin rpy="0 0 0" xyz="0 0 0"/>
+      <geometry>
+        <mesh filename="package://robominer_description/meshes/cuerpo.stl" scale="0.001 0.001 0.001"/>
+      </geometry>
+       <material name="silver"/>
+    </visual>
+    <collision>
+      <origin rpy="0 0 0" xyz="0 0 0"/>
+      <geometry>
+        <mesh filename="package://robominer_description/meshes/cuerpo.stl" scale="0.001 0.001 0.001"/>
+      </geometry>
+    </collision>
+  </link>
+  <xacro:macro name="body" params="parent child">
+    <joint name="fixed" type="fixed">
+      <origin rpy="0 0 0" xyz="0 0 0.1"/>
+      <parent link="${parent}"/>
+      <child link="${child}"/>
+    </joint>
+  </xacro:macro>
+>>>>>>> 7d42af75b2395a7bc20068cb95b739e23b31b89a
 </robot>

Commit message: Último commit

File: robominer_description/urdf/cuerpo.xacro (robot description, xacro)
@@ -1,5 +1,4 @@
 <?xml version="1.0" ?>
 <robot name="cuerpo" xmlns:xacro="http://www.ros.org/wiki/xacro">
-<<<<<<< HEAD
 <link name="cuerpo">
   <inertial>
@@ -73,32 +72,3 @@
 	</joint>
 </xacro:macro>
-=======
-  <link name="cuerpo">
-    <inertial>
-      <origin rpy="0 0 0" xyz="1.2607010642475455e-06 -1.9705023201073385e-17 0.030000000000039998"/>
-      <mass value="2"/>
-      <inertia ixx="0.155393" ixy="-0.0" ixz="-0.0" iyy="0.159826" iyz="-0.0" izz="0.297615"/>
-    </inertial>
-    <visual>
-      <origin rpy="0 0 0" xyz="0 0 0"/>
-      <geometry>
-        <mesh filename="package://robominer_description/meshes/cuerpo.stl" scale="0.001 0.001 0.001"/>
-      </geometry>
-       <material name="silver"/>
-    </visual>
-    <collision>
-      <origin rpy="0 0 0" xyz="0 0 0"/>
-      <geometry>
-        <mesh filename="package://robominer_description/meshes/cuerpo.stl" scale="0.001 0.001 0.001"/>
-      </geometry>
-    </collision>
-  </link>
-  <xacro:macro name="body" params="parent child">
-    <joint name="fixed" type="fixed">
-      <origin rpy="0 0 0" xyz="0 0 0.1"/>
-      <parent link="${parent}"/>
-      <child link="${child}"/>
-    </joint>
-  </xacro:macro>
->>>>>>> 7d42af75b2395a7bc20068cb95b739e23b31b89a
 </robot>
